File: shield/moros.kicad_pcb (KiCad board)
At the start: 2 copper layers, 48.3 x 18.3 mm, 7 parts, among them U1 ARDUINO_MICRO_SHIELD

Commit message: Clean up edges, prep files for OSHpark fab
Other:
- board size 48.3 x 18.3 mm -> 48.8 x 18.8 mm
